File: tests/input_samples/kibom-test.sch (KiCad schematic (older format))
At the start: 14 parts

Commit message: Fixed tests/input_samples/kibom-test.sch not synced with netlist
Parts:
- R6: Config (none) -> DNF
- R7: Config (none) -> DNC
Changed lines of the file:
@@
 F 2 "Resistor_SMD:R_0805_2012Metric" V 2130 3100 50  0001 C CNN
 F 3 "~" H 2200 3100 50  0001 C CNN
+F 4 "DNF" V 2200 3100 50  0001 C CNN "Config"
 	1    2200 3100
 	1    0    0    -1
@@
 F 2 "Resistor_SMD:R_0805_2012Metric" V 2430 3100 50  0001 C CNN
 F 3 "~" H 2500 3100 50  0001 C CNN
+F 4 "DNC" V 2500 3100 50  0001 C CNN "Config"
 	1    2500 3100
 	1    0    0    -1
