File: tests/input_samples/kibom-variante.sch (KiCad schematic (older format))
At the start: 20 parts

Commit message: Fixed isFixed (DNC)
Also added a couple of simple tests.
Parts:
- R19: Config bla bla DNF ble ble -> bla bla DNF ble DNC ble
- R2: Config -V2,-V3 -> -V2,-V3,DNC
Changed lines of the file:
@@
 F 2 "Resistor_SMD:R_0805_2012Metric" V 2430 2550 50  0001 C CNN
 F 3 "~" H 2500 2550 50  0001 C CNN
-F 4 "-V2,-V3" V 2500 2550 50  0001 C CNN "Config"
+F 4 "-V2,-V3,DNC" V 2500 2550 50  0001 C CNN "Config"
 	1    2500 2550
 	1    0    0    -1
@@
 F 2 "Resistor_SMD:R_0805_2012Metric" V 2680 4350 50  0001 C CNN
 F 3 "~" H 2750 4350 50  0001 C CNN
-F 4 "bla bla DNF ble ble" V 2750 4350 50  0001 C CNN "Config"
+F 4 "bla bla DNF ble DNC ble " V 2750 4350 50  0001 C CNN "Config"
 	1    2750 4350
 	1    0    0    -1
